File: pcb/DrikrAIO/hardware/DrikrAIO.kicad_pcb (KiCad board)
At the start: 6 copper layers, 50 x 50 mm, 347 parts, among them J601 5V, J602 5V, J603 5V, J604 5V, J606 5V, J607 5V, J609 5V, J610 5V, J611 5V, J613 5V, J614 5V, J615 5V, J616 5V, J617 5V, J618 5V, J620 5V, J621 5V, J622 5V, J623 5V, J624 5V, J625 5V, J627 5V, J629 5V, J631 5V, J632 5V, J633 5V, J634 5V, J635 5V, J636 5V, J637 5V, J639 5V, J640 5V, J641 5V, J649 5V, J801 SM08B-SRSS-TB, P601 SM08B-SRSS-TB(LF)(SN), Q101 AP1606, Q102 AP1606, Q1102 SP40N01GHNK, Q1107 SP40N01GHNK, Q1111 SP40N01GHNK, Q1113 SP40N01GHNK, Q1117 SP40N01GHNK, Q1120 SP40N01GHNK, Q1202 SP40N01GHNK, Q1207 SP40N01GHNK, Q1211 SP40N01GHNK, Q1213 SP40N01GHNK, Q1217 SP40N01GHNK, Q1220 SP40N01GHNK, Q1302 SP40N01GHNK, Q1307 SP40N01GHNK, Q1311 SP40N01GHNK, Q1313 SP40N01GHNK, Q1317 SP40N01GHNK, Q1320 SP40N01GHNK, Q1402 SP40N01GHNK, Q1407 SP40N01GHNK, Q1411 SP40N01GHNK, Q1413 SP40N01GHNK, Q1417 SP40N01GHNK, Q1420 SP40N01GHNK, U101 RP2354A, U102 TS2306A 240GF MSM 9_C2976675, U1101 NSG2065Q, U1108 AT32F421G8U7, U1201 NSG2065Q, U1208 AT32F421G8U7, U1301 NSG2065Q, U1308 AT32F421G8U7, U1401 NSG2065Q, U1408 AT32F421G8U7, U201 LP5912-1.8DRVR, U202 LMR51430YFDDCR, U203 LMR51430YFDDCR, U204 LP5912-3.3DRVR, U301 BMI270, U401 COS8051SOT, U402 SN74LVC1G3157DTBR, U403 TLV7031DPWR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

Commit message: DrikrAIO: placement optimisation -- no routing
Placement only. No tracks, no schematic change, no manufacturing outputs.

FREEZE NOTE, STATED RATHER THAN WORKED AROUND: placement necessarily changes
DrikrAIO.kicad_pcb, which is a hash-protected freeze artefact, so the freeze
broke by design and was re-taken at the new state. Every freeze ASSERTION still
holds -- 0 tracks, 0 vias, 8 netclasses, Phase/VBAT 6.6 mm, min_clearance 0.09,
MOSFET uncommitted, no manufacturing output. The electrical requirements were
not touched.

FOUR BLOCKS IN THE TASK DO NOT EXIST ON THIS BOARD and were not invented:
barometer, magnetometer, GPS interface and VTX are all absent from the design,
verified by search across every schematic. The VTX exists only as a gated 10 V
rail and a connector; there is no VTX to place, filter or heatsink.

SYMMETRY IS THE THERMAL DECISION. Airflow DIRECTION is an open requirement, so
the four ESC channels sit in identical quadrants and behave the same whichever
way the air moves. Within each quadrant parts are ordered MOSFETs, then gate
driver and channel MCU, then ceramics, and packed FROM THE OUTER CORNER INWARD
-- which puts the six FETs at the board edge where the airflow is under any
direction assumption, and lands the driver and local ceramics immediately
beside them for the commutation loop. All 24 MOSFETs and all 8 drivers/MCUs are
on the board.

IMU AT BOARD CENTRE. Every top-side position on a board this dense sits above
something; the question is what. The centre sits above the shunt and regulator
strip, which is a DC path rather than a switching node, and is the point
furthest from all four MOSFET clusters at once. RF and the FC switching
regulators went to opposite corners.

THREE ORDERING BUGS FOUND BY CHECKING RATHER THAN ASSUMING. Sorting non-ESC
bands alphabetically staged U701 -- the 2.4 GHz transceiver -- off the board
while keeping its decoupling on it. Rsense was absent from the priority table
entirely and defaulted last, so both 0.2 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
Parts:
- moved USB101 251.0 mm to (25.1, 4.04)
- moved U202 238.9 mm to (7.21, 3.86)
- moved U203 238.9 mm to (11.1, 3.86)
- moved U204 238.9 mm to (14.4, 3.54)
- moved U1308 204.9 mm to (9.45, 31.5)
- moved U1301 204.8 mm to (4.76, 31.4)
- moved U1408 199.8 mm to (40.6, 31.5)
- moved Q1420 198.7 mm to (32.0, 37.4)
- moved U1401 190.1 mm to (45.6, 31.4)
- moved Q1317 186.2 mm to (12.2, 37.4)
- moved Q1320 186.2 mm to (18.7, 37.4)
- moved Q1417 185.8 mm to (38.6, 37.4)
- moved U1108 151.7 mm to (9.45, 18.5)
- moved U1101 151.7 mm to (4.76, 18.5)
- moved U1208 146.6 mm to (40.6, 18.5)
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